Commit message: feat: add wheel links and joints to urdf

File: diffbot_description/urdf/diffbot.urdf.xacro (robot description, xacro)
@@ -2,10 +2,39 @@
 <!--diffbot with one link for now, just a box-->
 <robot name="diffbot">
+  <!--all the links first-->
   <link name="base_link">
     <visual>
       <geometry>
-        <box size="0.6 0.4 0.2"/>
+        <box size="0.4 0.6 0.2"/>
       </geometry>
     </visual>
   </link>
+  <!--the "height" of the wheels is the radius-->
+  <link name="left_wheel_link">
+    <visual>
+      <origin rpy="1.57079632679 0 0" xyz="0 0 0"/>
+      <geometry>
+        <cylinder length="0.01" radius="0.1"/>
+      </geometry>
+    </visual>
+  </link>
+  <link name="right_wheel_link">
+    <visual>
+      <origin rpy="1.57079632679 0 0" xyz="0 0 0"/>
+      <geometry>
+        <cylinder length="0.01" radius="0.1"/>
+      </geometry>
+    </visual>
+  </link>
+  <!--all the joints for the tf2 tree-->
+  <joint name="left_wheel_joint" type="continuous">
+    <parent link="base_link"/>
+    <child link="left_wheel_link"/>
+    <origin rpy="0 0 0" xyz="0 -0.2 -0.15"/>
+  </joint>
+  <joint name="right_wheel_joint" type="continuous">
+    <parent link="base_link"/>
+    <child link="right_wheel_link"/>
+    <origin rpy="0 0 0" xyz="0 0.2 -0.15"/>
+  </joint>
 </robot>

Commit message: feat: update urdf and switch to jsp gui

File: diffbot_description/urdf/diffbot.urdf.xacro (robot description, xacro)
@@ -1,40 +1,104 @@
-<?xml version="1.0"?>
-<!--diffbot with one link for now, just a box-->
+<?xml version='1.0'?>
 <robot name="diffbot">
-  <!--all the links first-->
   <link name="base_link">
     <visual>
+      <origin xyz="0 0 0" rpy="0 0 0"/>
       <geometry>
-        <box size="0.4 0.6 0.2"/>
+          <box size="0.5 0.5 0.25"/>
       </geometry>
+      <material name="blue">
+        <color rgba="0 0.5 1 1"/>
+      </material>
     </visual>
+    <collision>
+      <origin xyz="0 0 0" rpy="0 0 0"/>
+      <geometry>
+          <box size="0.5 0.5 0.25"/>
+      </geometry>
+    </collision>
+    <inertial>
+      <mass value="5"/>
+      <inertia ixx="0.13" ixy="0.0" ixz="0.0" iyy="0.21" iyz="0.0" izz="0.13"/>
+    </inertial>
   </link>
-  <!--the "height" of the wheels is the radius-->
+  <link name="caster_link">
+    <visual>
+      <origin xyz="0.0 0 0" rpy="0 0 0"/>
+      <geometry>
+        <sphere radius="0.05"/>
+      </geometry>
+      <material name="darkgray">
+        <color rgba=".2 .2 .2 1"/>
+      </material>
+    </visual>
+    <collision>
+      <origin xyz="0 0 0" rpy="0 0 0"/>
+      <geometry>
+        <sphere radius="0.05"/>
+      </geometry>
+    </collision>
+    <inertial>
+      <mass value="0.5"/>
+      <inertia ixx="0.0001" ixy="0.0" ixz="0.0" iyy="0.0001" iyz="0.0" izz="0.0001"/>
+    </inertial>
+  </link>
+  <joint name="caster_joint" type="fixed">
+    <parent link="base_link"/>
+    <child link="caster_link"/>
+    <origin xyz="0.2 0 -0.125" rpy="0 0 0"/>
+  </joint>
+  <link name="right_wheel_link">
+    <visual>
+      <origin xyz="0 0 0" rpy="1.570795 0 0"/>
+      <geometry>
+          <cylinder length="0.1" radius="0.2"/>
+      </geometry>
+      <material name="darkgray">
+        <color rgba=".2 .2 .2 1"/>
+      </material>
+    </visual>
+    <collision>
+      <origin xyz="0 0 0" rpy="1.570795 0 0"/>
+      <geometry>
+          <cylinder length="0.1" radius="0.2"/>
+      </geometry>
+    </collision>
+    <inertial>
+      <mass value="0.5"/>
+      <inertia ixx="0.01" ixy="0.0" ixz="0.0" iyy="0.005" iyz="0.0" izz="0.005"/>
+    </inertial>
+  </link>
+  <joint name="right_wheel_joint" type="continuous">
+    <parent link="base_link"/>
+    <child link="right_wheel_link"/>
+    <origin xyz="0 -0.30 0" rpy="0 0 0"/>
+    <axis xyz="0 1 0"/>
+  </joint>
   <link name="left_wheel_link">
     <visual>
-      <origin rpy="1.57079632679 0 0" xyz="0 0 0"/>
+      <origin xyz="0 0 0" rpy="1.570795 0 0"/>
       <geometry>
-        <cylinder length="0.01" radius="0.1"/>
+          <cylinder length="0.1" radius="0.2"/>
       </geometry>
+      <material name="darkgray">
+        <color rgba=".2 .2 .2 1"/>
+      </material>
     </visual>
+    <collision>
+      <origin xyz="0 0 0" rpy="1.570795 0 0"/>
+      <geometry>
+          <cylinder length="0.1" radius="0.2"/>
+      </geometry>
+    </collision>
+    <inertial>
+      <mass value="0.5"/>
+      <inertia ixx="0.01" ixy="0.0" ixz="0.0" iyy="0.005" iyz="0.0" izz="0.005"/>
+    </inertial>
   </link>
-  <link name="right_wheel_link">
-    <visual>
-      <origin rpy="1.57079632679 0 0" xyz="0 0 0"/>
-      <geometry>
-        <cylinder length="0.01" radius="0.1"/>
-      </geometry>
-    </visual>
-  </link>
-  <!--all the joints for the tf2 tree-->
   <joint name="left_wheel_joint" type="continuous">
     <parent link="base_link"/>
     <child link="left_wheel_link"/>
-    <origin rpy="0 0 0" xyz="0 -0.2 -0.15"/>
-  </joint>
-  <joint name="right_wheel_joint" type="continuous">
-    <parent link="base_link"/>
-    <child link="right_wheel_link"/>
-    <origin rpy="0 0 0" xyz="0 0.2 -0.15"/>
+    <origin xyz="0 0.30 0" rpy="0 0 0"/>
+    <axis xyz="0 1 0"/>
   </joint>
 </robot>

Commit message: feat: modularise urdf

File: diffbot_description/urdf/diffbot.urdf.xacro (robot description, xacro)
@@ -1,104 +1,5 @@
-<?xml version='1.0'?>
-<robot name="diffbot">
-  <link name="base_link">
-    <visual>
-      <origin xyz="0 0 0" rpy="0 0 0"/>
-      <geometry>
-          <box size="0.5 0.5 0.25"/>
-      </geometry>
-      <material name="blue">
-        <color rgba="0 0.5 1 1"/>
-      </material>
-    </visual>
-    <collision>
-      <origin xyz="0 0 0" rpy="0 0 0"/>
-      <geometry>
-          <box size="0.5 0.5 0.25"/>
-      </geometry>
-    </collision>
-    <inertial>
-      <mass value="5"/>
-      <inertia ixx="0.13" ixy="0.0" ixz="0.0" iyy="0.21" iyz="0.0" izz="0.13"/>
-    </inertial>
-  </link>
-  <link name="caster_link">
-    <visual>
-      <origin xyz="0.0 0 0" rpy="0 0 0"/>
-      <geometry>
-        <sphere radius="0.05"/>
-      </geometry>
-      <material name="darkgray">
-        <color rgba=".2 .2 .2 1"/>
-      </material>
-    </visual>
-    <collision>
-      <origin xyz="0 0 0" rpy="0 0 0"/>
-      <geometry>
-        <sphere radius="0.05"/>
-      </geometry>
-    </collision>
-    <inertial>
-      <mass value="0.5"/>
-      <inertia ixx="0.0001" ixy="0.0" ixz="0.0" iyy="0.0001" iyz="0.0" izz="0.0001"/>
-    </inertial>
-  </link>
-  <joint name="caster_joint" type="fixed">
-    <parent link="base_link"/>
-    <child link="caster_link"/>
-    <origin xyz="0.2 0 -0.125" rpy="0 0 0"/>
-  </joint>
-  <link name="right_wheel_link">
-    <visual>
-      <origin xyz="0 0 0" rpy="1.570795 0 0"/>
-      <geometry>
-          <cylinder length="0.1" radius="0.2"/>
-      </geometry>
-      <material name="darkgray">
-        <color rgba=".2 .2 .2 1"/>
-      </material>
-    </visual>
-    <collision>
-      <origin xyz="0 0 0" rpy="1.570795 0 0"/>
-      <geometry>
-          <cylinder length="0.1" radius="0.2"/>
-      </geometry>
-    </collision>
-    <inertial>
-      <mass value="0.5"/>
-      <inertia ixx="0.01" ixy="0.0" ixz="0.0" iyy="0.005" iyz="0.0" izz="0.005"/>
-    </inertial>
-  </link>
-  <joint name="right_wheel_joint" type="continuous">
-    <parent link="base_link"/>
-    <child link="right_wheel_link"/>
-    <origin xyz="0 -0.30 0" rpy="0 0 0"/>
-    <axis xyz="0 1 0"/>
-  </joint>
-  <link name="left_wheel_link">
-    <visual>
-      <origin xyz="0 0 0" rpy="1.570795 0 0"/>
-      <geometry>
-          <cylinder length="0.1" radius="0.2"/>
-      </geometry>
-      <material name="darkgray">
-        <color rgba=".2 .2 .2 1"/>
-      </material>
-    </visual>
-    <collision>
-      <origin xyz="0 0 0" rpy="1.570795 0 0"/>
-      <geometry>
-          <cylinder length="0.1" radius="0.2"/>
-      </geometry>
-    </collision>
-    <inertial>
-      <mass value="0.5"/>
-      <inertia ixx="0.01" ixy="0.0" ixz="0.0" iyy="0.005" iyz="0.0" izz="0.005"/>
-    </inertial>
-  </link>
-  <joint name="left_wheel_joint" type="continuous">
-    <parent link="base_link"/>
-    <child link="left_wheel_link"/>
-    <origin xyz="0 0.30 0" rpy="0 0 0"/>
-    <axis xyz="0 1 0"/>
-  </joint>
+<?xml version="1.0"?>
+<robot name="diffbot" xmlns:xacro="http://www.ros.org/wiki/xacro">
+    <xacro:include filename="common_properties.xacro" />
+    <xacro:include filename="mobile_base.xacro" />
 </robot>
