Commit message: feat: move frictions to collision surface in core xacro, add gazebo ros2control plugin

File: diffbot_description/urdf/diffbot.core.xacro (robot description, xacro)
@@ -1,4 +1,11 @@
 <?xml version="1.0"?>
 <robot xmlns:xacro="http://www.ros.org/wiki/xacro">
+    <!--Materials-->
+    <material name="blue">
+        <color rgba="0 0 0.5 1" />
+    </material>
+    <material name="grey">
+        <color rgba="0.5 0.5 0.5 1" />
+    </material>
     <!--Dimensions-->
     <xacro:property name="base_length" value="0.6" />
@@ -77,4 +84,12 @@
                 </geometry>
                 <origin xyz="0 0 0" rpy="${pi / 2.0} 0 0" />
+                <surface>
+                    <friction>
+                        <ode>
+                            <mu>1.0</mu>
+                            <mu2>1.0</mu2>
+                        </ode>
+                    </friction>
+                </surface>
             </collision>
             <xacro:inertial_cylinder mass="${wheel_mass}" radius="${wheel_radius}" length="${wheel_length}" />
@@ -91,10 +106,18 @@
             <material name="grey" />
         </visual>
-         <visual>
+         <collision>
             <geometry>
                 <sphere radius="${wheel_radius / 2.0}" />
             </geometry>
             <origin xyz="0 0 0" rpy="0 0 0" />
-        </visual>
+            <surface>
+                <friction>
+                    <ode>
+                        <mu>0.1</mu>
+                        <mu2>0.1</mu2>
+                    </ode>
+                </friction>
+            </surface>
+        </collision>
         <xacro:inertial_sphere mass="${caster_mass}" radius="${wheel_radius / 2.0}" />
     </link>

File: diffbot_description/urdf/diffbot.urdf.xacro (robot description, xacro)
@@ -1,5 +1,5 @@
 <?xml version="1.0"?>
 <robot name="diffbot" xmlns:xacro="http://www.ros.org/wiki/xacro">
-    <xacro:include filename="common_properties.xacro" />
-    <xacro:include filename="mobile_base.xacro" />
+    <xacro:include filename="diffbot.core.xacro" />
+    <xacro:include filename="diffbot.ros2_control.xacro" />
 </robot>
