Commit message: feat: ros2control

File: diffbot_description/urdf/diffbot.ros2_control.xacro (robot description, xacro)
@@ -1,3 +1,27 @@
 <?xml version="1.0"?>
 <robot xmlns:xacro="http://www.ros.org/wiki/xacro">
+    <ros2_control name="DiffBotSystem" type="system">
+        <!-- Hardware plugin for Gazebo (Ignition) -->
+        <hardware>
+            <plugin>gz_ros2_control/GazeboSimSystem</plugin>
+        </hardware>
+        <!-- Left wheel joint -->
+        <joint name="base_left_wheel_joint">
+            <command_interface name="velocity">
+                <param name="min">-10</param>
+                <param name="max">10</param>
+            </command_interface>
+            <state_interface name="position"/>
+            <state_interface name="velocity"/>
+        </joint>
+        <!-- Right wheel joint -->
+        <joint name="base_right_wheel_joint">
+            <command_interface name="velocity">
+                <param name="min">-10</param>
+                <param name="max">10</param>
+            </command_interface>
+            <state_interface name="position"/>
+            <state_interface name="velocity"/>
+        </joint>
+    </ros2_control>
 </robot>

File: diffbot_description/urdf/diffbot.urdf.xacro (robot description, xacro)
@@ -2,4 +2,5 @@
 <robot name="diffbot" xmlns:xacro="http://www.ros.org/wiki/xacro">
     <xacro:include filename="diffbot.core.xacro" />
+    <xacro:include filename="diffbot.gazebo.xacro" />
     <xacro:include filename="diffbot.ros2_control.xacro" />
 </robot>
